Commit message: fix:根据车体新模型修改了urdf文件，同时加上了note笔记部分

File: sentry_description/urdf/mas2027_sentry.urdf (robot description, URDF)
Before this commit: robot mas2027_sentry, 5 links, 4 joints
Links:
- removed link lakibeam_frame
Joints:
- removed joint lakibeam_joint
- joint lidar_joint: origin xyz=0.09 0.03 0.11 rpy=0.3572 0 1.5708 -> xyz=0.00 -0.15 0.11 rpy=0.8389 0 0

Commit message: feat:新增nav导航同时修复urdf模型和mid360驱动重力方向参数

File: sentry_description/urdf/mas2027_sentry.urdf (robot description, URDF)
Before this commit: robot mas2027_sentry, 4 links, 3 joints
Joints:
- joint lidar_joint: origin xyz=0.00 -0.15 0.11 rpy=0.8389 0 0 -> xyz=0.00 0.15 0.11 rpy=-0.8389 0 0
